File: pcb/onyks-iot-monitor-weather-pcb/old_bad.kicad_pcb (KiCad board)
At the start: 2 copper layers, 100 x 100 mm, 25 parts, among them J1 53398-0371, J10 Conn_01x02_Pin, J2 53398-0371, J3 53048-0810, J4 53398-0371, J5 53398-0371, J6 53398-0371, J7 53398-0371, J8 53398-0371, J9 53398-0371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

Commit message: Added PCBv1.0
Routing:
- net /IO0: track 137.0 -> 111.9 mm
- net /DHT22: track 50.8 -> 37.0 mm
- net GND: track 256.8 -> 266.4 mm
Changed lines of the file:
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@@
 	)
 	(segment
-		(start 133 68.7)
-		(end 133 62.5)
+		(start 127.5 99)
+		(end 127 99.5)
 		(width 0.2)
 		(layer "F.Cu")
@@
 	)
 	(segment
+		(start 128.8 99)
+		(end 127.5 99)
+		(width 0.2)
+		(layer "F.Cu")
+		(net 1)
+	)
+	(segment
 		(start 112.835 80.165)
 		(end 114 79)
@@
 	)
 	(segment
-		(start 133.8 96.3)
-		(end 133.8 99.45)
-		(width 0.2)
-		(layer "F.Cu")
-		(net 1)
-	)
-	(segment
-		(start 133 68.7)
-		(end 133 95.5)
-		(width 0.2)
-		(layer "F.Cu")
-		(net 1)
-	)
-	(segment
 		(start 144.68 63.68)
 		(end 144 63)
@@
 	)
 	(segment
-		(start 132.75 61)
-		(end 132.75 62.25)
+		(start 133 68.7)
+		(end 133 94.8)
 		(width 0.2)
 		(layer "F.Cu")
@@
 	)
 	(segment
+		(start 133.8 106.2)
+		(end 133.8 99.45)
+		(width 0.2)
+		(layer "F.Cu")
+		(net 1)
+	)
+	(segment
 		(start 140.5 63.025)
 		(end 141.155 63.68)
@@
 	)
 	(segment
+		(start 133.5 106.5)
+		(end 133.8 106.2)
+		(width 0.2)
+		(layer "F.Cu")
+		(net 1)
+	)
+	(segment
+		(start 127.5 106.5)
+		(end 133.5 106.5)
+		(width 0.2)
+		(layer "F.Cu")
+		(net 1)
+	)
+	(segment
 		(start 160 82.1)
 		(end 160.9 82.1)
@@
 	)
 	(segment
-		(start 133 95.5)
-		(end 133.8 96.3)
-		(width 0.2)
-		(layer "F.Cu")
-		(net 1)
-	)
-	(segment
 		(start 110.5 64.5)
 		(end 111 64)
@@
 	)
 	(segment
+		(start 127 106)
+		(end 127.5 106.5)
+		(width 0.2)
+		(layer "F.Cu")
+		(net 1)
+	)
+	(segment
 		(start 112.5 57.5)
 		(end 111.5 57.5)
@@
 	)
 	(segment
+		(start 133 94.8)
+		(end 128.8 99)
+		(width 0.2)
+		(layer "F.Cu")
+		(net 1)
+	)
+	(segment
 		(start 113.2 58.2)
 		(end 112.5 57.5)
@@
 	)
 	(segment
-		(start 132.75 62.25)
-		(end 133 62.5)
-		(width 0.2)
-		(layer "F.Cu")
-		(net 1)
-	)
-	(segment
 		(start 113.2 59.7)
 		(end 115.405 57.495)
@@
 		(net 1)
 	)
+	(segment
+		(start 127 99.5)
+		(end 127 106)
+		(width 0.2)
+		(layer "F.Cu")
+		(net 1)
+	)
 	(via
 		(at 111.5 57.5)
@@
 	)
 	(segment
-		(start 138.5 63.5)
-		(end 135.5 63.5)
-		(width 0.2)
-		(layer "B.Cu")
-		(net 1)
-	)
-	(segment
 		(start 167.5 88.5)
 		(end 183.5 88.5)
@@
 	)
 	(segment
-		(start 135.5 63.5)
-		(end 134.5 62.5)
-		(width 0.2)
-		(layer "B.Cu")
-		(net 1)
-	)
-	(segment
-		(start 134.5 62.5)
-		(end 133 62.5)
-		(width 0.2)
-		(layer "B.Cu")
-		(net 1)
-	)
-	(segment
 		(start 163.75 84.75)
 		(end 163.5 84.5)
@@
 	)
 	(segment
+		(start 149 77)
+		(end 149 74)
+		(width 0.2)
+		(layer "F.Cu")
+		(net 18)
+	)
+	(segment
+		(start 144 92)
+		(end 144 82)
+		(width 0.2)
+		(layer "F.Cu")
+		(net 18)
+	)
+	(segment
+		(start 149.005 74.005)
+		(end 150.5 74.005)
+		(width 0.2)
+		(layer "F.Cu")
+		(net 18)
+	)
+	(segment
+		(start 132.5 98)
+		(end 133 97.5)
+		(width 0.2)
+		(layer "F.Cu")
+		(net 18)
+	)
+	(segment
+		(start 133 97.5)
+		(end 138.5 97.5)
+		(width 0.2)
+		(layer "F.Cu")
+		(net 18)
+	)
+	(segment
+		(start 138.5 97.5)
+		(end 144 92)
+		(width 0.2)
+		(layer "F.Cu")
+		(net 18)
+	)
+	(segment
+		(start 144 82)
+		(end 149 77)
+		(width 0.2)
+		(layer "F.Cu")
+		(net 18)
+	)
+	(segment
 		(start 149 74)
 		(end 149.005 74.005)
@@
 	)
 	(segment
-		(start 132.55 99.45)
-		(end 132.55 104.55)
-		(width 0.2)
-		(layer "F.Cu")
-		(net 18)
-	)
-	(segment
-		(start 149.005 74.005)
-		(end 150.5 74.005)
-		(width 0.2)
-		(layer "F.Cu")
-		(net 18)
-	)
-	(segment
-		(start 133 105)
-		(end 142.5 105)
-		(width 0.2)
-		(layer "F.Cu")
-		(net 18)
-	)
-	(segment
-		(start 149 77)
-		(end 149 74)
-		(width 0.2)
-		(layer "F.Cu")
-		(net 18)
-	)
-	(segment
-		(start 132.55 104.55)
-		(end 133 105)
-		(width 0.2)
-		(layer "F.Cu")
-		(net 18)
-	)
-	(segment
-		(start 142.5 105)
-		(end 144 103.5)
-		(width 0.2)
-		(layer "F.Cu")
-		(net 18)
-	)
-	(segment
-		(start 144 103.5)
-		(end 144 82)
-		(width 0.2)
-		(layer "F.Cu")
-		(net 18)
-	)
-	(segment
-		(start 144 82)
-		(end 149 77)
-		(width 0.2)
-		(layer "F.Cu")
-		(net 18)
-	)
-	(segment
 		(start 132.55 99.2)
 		(end 132.5 99.15)
@@
 	)
 	(segment
+		(start 132.5 99.15)
+		(end 132.5 98)
+		(width 0.2)
+		(layer "F.Cu")
+		(net 18)
+	)
+	(segment
 		(start 132.55 99.45)
 		(end 132.55 99.2)
@@
 	)
 	(segment
-		(start 195.5 72.5)
-		(end 193.995 74.005)
+		(start 127.5 112.5)
+		(end 139.5 112.5)
 		(width 0.2)
 		(layer "F.Cu")
@@
 	)
 	(segment
-		(start 172 80)
-		(end 172 74.005)
+		(start 126 111)
+		(end 127.5 112.5)
+		(width 0.2)
+		(layer "F.Cu")
+		(net 37)
+	)
+	(segment
+		(start 139.5 112.5)
+		(end 172 80)
+		(width 0.2)
+		(layer "F.Cu")
+		(net 37)
+	)
+	(segment
+		(start 116.5875 78.4125)
+		(end 126 87.825)
+		(width 0.2)
+		(layer "F.Cu")
+		(net 37)
+	)
+	(segment
+		(start 113.475 80.5)
+		(end 114.5 80.5)
 		(width 0.2)
 		(layer "F.Cu")
@@
 	)
 	(segment
-		(start 172 74.005)
+		(start 169.505 74.005)
 		(end 168 74.005)
 		(width 0.2)
@@
 	)
 	(segment
-		(start 193.995 74.005)
-		(end 172 74.005)
+		(start 172 76.5)
+		(end 169.505 74.005)
 		(width 0.2)
 		(layer "F.Cu")
@@
 	)
 	(segment
-		(start 118.675 80.5)
-		(end 126 87.825)
+		(start 114.5 80.5)
+		(end 116.5875 78.4125)
 		(width 0.2)
 		(layer "F.Cu")
@@
 	)
 	(segment
-		(start 114.5 80.5)
-		(end 118.675 80.5)
+		(start 172 80)
+		(end 172 76.5)
 		(width 0.2)
 		(layer "F.Cu")
@@
 	)
 	(segment
-		(start 139.5 112.5)
-		(end 172 80)
-		(width 0.2)
-		(layer "F.Cu")
-		(net 37)
-	)
-	(segment
-		(start 114.625 80.375)
-		(end 114.5 80.5)
-		(width 0.2)
-		(layer "F.Cu")
-		(net 37)
-	)
-	(segment
-		(start 113.475 80.5)
-		(end 114.5 80.5)
-		(width 0.2)
-		(layer "F.Cu")
-		(net 37)
-	)
-	(segment
-		(start 127.5 112.5)
-		(end 139.5 112.5)
-		(width 0.2)
-		(layer "F.Cu")
-		(net 37)
-	)
-	(segment
 		(start 114.625 76.45)
-		(end 114.625 80.375)
-		(width 0.2)
-		(layer "F.Cu")
-		(net 37)
-	)
-	(segment
-		(start 126 111)
-		(end 127.5 112.5)
+		(end 116.5875 78.4125)
 		(width 0.2)
 		(layer "F.Cu")
@@
 	(segment
 		(start 116.5 75.5)
+		(end 117 75)
+		(width 0.2)
+		(layer "F.Cu")
+		(net 38)
+	)
+	(segment
+		(start 117 75)
+		(end 117 73)
+		(width 0.2)
+		(layer "F.Cu")
+		(net 38)
+	)
+	(segment
+		(start 117 73)
 		(end 116.5 72.5)
 		(width 0.2)
@@
 	)
 	(segment
-		(start 123.5 83.04)
+		(start 115 91.54)
+		(end 124 82.54)
+		(width 0.2)
+		(layer "B.Cu")
+		(net 39)
+	)
+	(segment
+		(start 124 77.5)
 		(end 123.5 77)
 		(width 0.2)
@@
 	)
 	(segment
-		(start 115 91.54)
-		(end 123.5 83.04)
-		(width 0.2)
-		(layer "B.Cu")
+		(start 124 82.54)
+		(end 124 77.5)
+		(width 0.2)
+		(layer "B.Cu")
