File: pcb/Programming.kicad_sch (KiCad schematic)
At the start: 6 parts, among them J11 Conn_01x06_Pin, J12 Conn_02x05_Odd_Even, Q1 SS8050, Q2 SS8050

Commit message: Drobne poprawki w schemacie elektrycznym
Parts:
- added C1, C2: 0.1uF/4VDC, Capacitor_SMD:C_0603_1608Metric, symbol Device:C
- added S3, S4: PTS636_SK25F_SMTR_LFS, 1bmoje:PTS636SK25FSMTRLFS, symbol Switch:SW_Push
Connections:
- net GND: now also C1.1, C2.1, S3.1, S4.1
- net UART_EN: now also C2.2, S4.2
- net UART_IO0: now also C1.2, S3.2
Other:
- note added: "Buttons for RESET and programming"
